File: door.sch (EAGLE design)
At the start: 11 parts, among them IC1 ATMEGA8-PU

Commit message: bigger pads
Parts:
- C1: value 10NF -> 10nf
- IC2: value (none) -> 5.0
- IC3: value (none) -> 3.3
- renumbered 10NF to C1, PIR to JP1, VREG3.3 to IC3, VREG5.0 to IC2
Connections:
- net GND: now also JP1.GND; no longer JP1.2
- net N$1: now also JP1.OUT; no longer JP1.1
- net N$6: now also JP1.VCC; no longer JP1.3
Changed lines of the file:
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@@
 <parts>
 <part name="IC1" library="atmega8" deviceset="ATMEGA8-PU" device=""/>
-<part name="VREG5.0" library="SparkFun" deviceset="V_REG_78XX" device="SINK"/>
-<part name="VREG3.3" library="SparkFun" deviceset="V_REG_78XX" device="SINK"/>
 <part name="BATTERY" library="SparkFun" deviceset="VCC" device=""/>
 <part name="SUPPLY1" library="supply2" deviceset="GND" device=""/>
-<part name="10NF" library="capacitor-wima" deviceset="C" device="2.5/4" value="10NF"/>
-<part name="PIR" library="SparkFun" deviceset="M03" device="PTH"/>
 <part name="G1" library="battery" deviceset="AB9V" device=""/>
 <part name="S1" library="switch-reed" deviceset="REED-SWITCH-" device="MK6-6"/>
@@
 <part name="LED2" library="led" deviceset="LED" device="3MM"/>
 <part name="JP2" library="SparkFun" deviceset="ARDUINO_SERIAL_PROGRAM" device="LONGPADS"/>
+<part name="IC2" library="SparkFun" deviceset="V_REG_78XX" device="SINK" value="5.0"/>
+<part name="IC3" library="SparkFun" deviceset="V_REG_78XX" device="SINK" value="3.3"/>
+<part name="C1" library="capacitor-wima" deviceset="C" device="2.5/4" value="10nf"/>
+<part name="JP1" library="SparkFun" deviceset="M03" device="PTH"/>
 </parts>
 <sheets>
@@
 <instances>
 <instance part="IC1" gate="1" x="71.12" y="15.24"/>
-<instance part="VREG5.0" gate="G$1" x="-10.16" y="68.58" rot="MR0"/>
-<instance part="VREG3.3" gate="G$1" x="20.32" y="68.58"/>
 <instance part="BATTERY" gate="1" x="-30.48" y="76.2"/>
 <instance part="SUPPLY1" gate="GND" x="0" y="-50.8"/>
-<instance part="10NF" gate="G$1" x="33.02" y="0"/>
-<instance part="PIR" gate="G$1" x="66.04" y="-48.26" rot="R180"/>
 <instance part="G1" gate="G$1" x="2.54" y="55.88" rot="R90"/>
 <instance part="S1" gate="G$1" x="68.58" y="-27.94" rot="R90"/>
@@
 <instance part="LED2" gate="G$1" x="68.58" y="-38.1" rot="R270"/>
 <instance part="JP2" gate="G$1" x="127" y="81.28" rot="MR270"/>
+<instance part="IC2" gate="G$1" x="-10.16" y="68.58" rot="MR0"/>
+<instance part="IC3" gate="G$1" x="20.32" y="68.58"/>
+<instance part="C1" gate="G$1" x="33.02" y="0"/>
+<instance part="JP1" gate="G$1" x="66.04" y="-48.26" rot="R180"/>
 </instances>
 <busses>
@@
 <wire x1="-30.48" y1="73.66" x2="5.08" y2="73.66" width="0.1524" layer="91"/>
 <wire x1="5.08" y1="73.66" x2="5.08" y2="68.58" width="0.1524" layer="91"/>
-<pinref part="VREG3.3" gate="G$1" pin="IN"/>
 <wire x1="5.08" y1="68.58" x2="12.7" y2="68.58" width="0.1524" layer="91"/>
-<pinref part="VREG5.0" gate="G$1" pin="IN"/>
 <wire x1="-2.54" y1="68.58" x2="2.54" y2="68.58" width="0.1524" layer="91"/>
 <pinref part="G1" gate="G$1" pin="+"/>
 <wire x1="2.54" y1="68.58" x2="5.08" y2="68.58" width="0.1524" layer="91"/>
 <junction x="2.54" y="68.58"/>
+<pinref part="IC2" gate="G$1" pin="IN"/>
+<pinref part="IC3" gate="G$1" pin="IN"/>
 </segment>
 </net>
@@
 <wire x1="33.02" y1="-12.7" x2="33.02" y2="-7.62" width="0.1524" layer="91"/>
 <wire x1="60.96" y1="-27.94" x2="0" y2="-27.94" width="0.1524" layer="91"/>
-<pinref part="PIR" gate="G$1" pin="2"/>
 <wire x1="58.42" y1="-48.26" x2="38.1" y2="-48.26" width="0.1524" layer="91"/>
 <wire x1="38.1" y1="-48.26" x2="0" y2="-48.26" width="0.1524" layer="91"/>
 <wire x1="38.1" y1="-50.8" x2="38.1" y2="-48.26" width="0.1524" layer="91"/>
 <wire x1="38.1" y1="-50.8" x2="40.64" y2="-50.8" width="0.1524" layer="91"/>
-<pinref part="10NF" gate="G$1" pin="2"/>
 <wire x1="33.02" y1="-5.08" x2="33.02" y2="-7.62" width="0.1524" layer="91"/>
-<pinref part="VREG5.0" gate="G$1" pin="GND"/>
 <wire x1="-10.16" y1="60.96" x2="-10.16" y2="35.56" width="0.1524" layer="91"/>
 <wire x1="-10.16" y1="35.56" x2="0" y2="35.56" width="0.1524" layer="91"/>
 <wire x1="0" y1="35.56" x2="2.54" y2="35.56" width="0.1524" layer="91"/>
-<pinref part="VREG3.3" gate="G$1" pin="GND"/>
 <wire x1="2.54" y1="35.56" x2="20.32" y2="35.56" width="0.1524" layer="91"/>
 <wire x1="20.32" y1="58.42" x2="20.32" y2="60.96" width="0.1524" layer="91"/>
@@
 <pinref part="JP2" gate="G$1" pin="GND"/>
 <wire x1="119.38" y1="58.42" x2="119.38" y2="76.2" width="0.1524" layer="91"/>
+<pinref part="IC2" gate="G$1" pin="GND"/>
+<pinref part="IC3" gate="G$1" pin="GND"/>
+<pinref part="C1" gate="G$1" pin="2"/>
+<pinref part="JP1" gate="G$1" pin="GND"/>
 </segment>
 </net>
@@
 <net name="N$1" class="0">
 <segment>
-<pinref part="VREG5.0" gate="G$1" pin="OUT"/>
 <wire x1="-17.78" y1="68.58" x2="-25.4" y2="68.58" width="0.1524" layer="91"/>
 <wire x1="-25.4" y1="68.58" x2="-25.4" y2="-45.72" width="0.1524" layer="91"/>
-<pinref part="PIR" gate="G$1" pin="1"/>
 <wire x1="58.42" y1="-45.72" x2="-25.4" y2="-45.72" width="0.1524" layer="91"/>
+<pinref part="IC2" gate="G$1" pin="OUT"/>
+<pinref part="JP1" gate="G$1" pin="OUT"/>
 </segment>
 </net>
@@
 <net name="N$6" class="0">
 <segment>
-<pinref part="PIR" gate="G$1" pin="3"/>
 <wire x1="58.42" y1="-50.8" x2="58.42" y2="-55.88" width="0.1524" layer="91"/>
 <wire x1="58.42" y1="-55.88" x2="106.68" y2="-55.88" width="0.1524" layer="91"/>
@@
 <wire x1="50.8" y1="-50.8" x2="58.42" y2="-50.8" width="0.1524" layer="91"/>
 <pinref part="R2" gate="G$1" pin="2"/>
+<pinref part="JP1" gate="G$1" pin="VCC"/>
+<junction x="58.42" y="-50.8"/>
 </segment>
 </net>
@@
 <segment>
 <pinref part="IC1" gate="1" pin="AVCC"/>
-<pinref part="VREG3.3" gate="G$1" pin="OUT"/>
 <wire x1="27.94" y1="68.58" x2="33.02" y2="68.58" width="0.1524" layer="91"/>
 <wire x1="33.02" y1="68.58" x2="33.02" y2="55.88" width="0.1524" layer="91"/>
@@
 <wire x1="40.64" y1="5.08" x2="33.02" y2="5.08" width="0.1524" layer="91"/>
 <wire x1="33.02" y1="5.08" x2="33.02" y2="7.62" width="0.1524" layer="91"/>
-<pinref part="10NF" gate="G$1" pin="1"/>
 <wire x1="33.02" y1="2.54" x2="33.02" y2="5.08" width="0.1524" layer="91"/>
 <pinref part="JP2" gate="G$1" pin="VCC"/>
 <wire x1="124.46" y1="55.88" x2="124.46" y2="76.2" width="0.1524" layer="91"/>
+<pinref part="IC3" gate="G$1" pin="OUT"/>
+<pinref part="C1" gate="G$1" pin="1"/>
 </segment>
 </net>
